File: Lab_Sensor_Version_1/Lab_Sensor_Version_1.kicad_sch (KiCad schematic)
At the start: 28 parts, among them U1 ESP32-POE, U2 AM2302, U3 SSD1306, U4 INMP441

Commit message: Fixing Version History
Parts:
- removed U1: ESP32-POE, ESP32-POE:MODULE_ESP32-POE, symbol ESP32-POE:ESP32-POE
- added U1: ESP32-POE, Custom_Parts:ESP32-POE, symbol Custom_Parts:ESP32-POE
- D1, D2, D3, D4, D5, D6: footprint Standard_LED_Throughhole:Standard_LED_Throughhole -> Custom_Parts:Standard_LED_Throughhole
- TP1, TP2: footprint 5002:KEYSTONE_5002 -> Custom_Parts:5002; symbol 5002:5002 -> Custom_Parts:5002
- U3: footprint SSD1306:128x64OLED -> Custom_Parts:SSD1306
- U4: footprint Custom_Footprints:INMP441 -> Custom_Parts:INMP441
Connections:
- net +3.3V: now also U4.2 (VDD), U1.EXT1_2 (+3.3V); no longer U4.4 (VDD)
- net GND: now also U4.3 (GND), U1.EXT1_3 (GND); no longer U4.6 (GND)
- net at R3.2: now also U1.EXT1_7 (GPIO2)
- net at R9.1: now also U4.1 (SO); no longer U4.2 (SD)
- net at R9.2: now also U1.EXT2_8 (GPIO15)
- net at R6.2: now also U1.EXT1_10 (GPIO5)
- net at R7.2: now also U1.EXT2_10 (GPIO13)
- net at TP1.TP: now also U1.EXT2_3 (GPI35)
- net at R8.2: now also U1.EXT2_9 (GPIO14)
- net at R12.1: now also U1.EXT2_5 (GPIO33)
- net at R10.1: now also U4.6 (SCK); no longer U4.1 (SCK)
- net at R10.2: now also U1.EXT2_7 (GPIO16)
- net at R4.2: now also U1.EXT1_8 (GPIO3)
- net at R2.2: now also U1.EXT1_6 (GPIO1)
- net at R1.2: now also U1.EXT1_5 (GPIO0)
- net at R11.2: now also U4.5 (SW); no longer U4.3 (SW)
- net at TP2.TP: now also U1.EXT2_2 (GPI36)
- net at R5.2: now also U1.EXT1_9 (GPIO4)
- net at R11.1: now also U1.EXT2_6 (GPIO32)
Other:
- moved on the sheet: C1, D1, D2, D3, D4, D5, D6, R1, R10, R11, R12, R13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
