File: Lab_Sensor_Version_1/Lab_Sensor_Version_1.kicad_sch (KiCad schematic)
At the start: 28 parts, among them U1 ESP32-POE, U2 AM2302, U3 SSD1306, U4 INMP441

Commit message: Rerouted 4 GPIO expanders
Connections:
- net at R7.2: now also U1.EXT1_8 (GPIO3); no longer U1.EXT1_10 (GPIO5)
- net at TP1.TP: now also U1.EXT1_10 (GPIO5); no longer U1.EXT1_8 (GPIO3)
- net at R8.2: now also U1.EXT1_7 (GPIO2); no longer U1.EXT1_9 (GPIO4)
- net at TP2.TP: now also U1.EXT1_9 (GPIO4); no longer U1.EXT1_7 (GPIO2)
Other:
- moved on the sheet: R7, R8, TP1, TP2
Changed lines of the file:
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@@
-	(wire
-		(pts
-			(xy 153.67 67.31) (xy 160.02 67.31)
-		)
-		(stroke
-			(width 0)
-			(type default)
-		)
-	)
 	(wire
 		(pts
@@
 	(wire
 		(pts
-			(xy 163.83 69.85) (xy 163.83 119.38)
-		)
-		(stroke
-			(width 0)
-			(type default)
-		)
-	)
-	(wire
-		(pts
 			(xy 91.44 100.33) (xy 91.44 106.68)
 		)
@@
 	(wire
 		(pts
+			(xy 160.02 62.23) (xy 160.02 124.46)
+		)
+		(stroke
+			(width 0)
+			(type default)
+		)
+	)
+	(wire
+		(pts
 			(xy 80.01 77.47) (xy 80.01 82.55)
 		)
@@
 	(wire
 		(pts
-			(xy 153.67 69.85) (xy 163.83 69.85)
-		)
-		(stroke
-			(width 0)
-			(type default)
-		)
-	)
-	(wire
-		(pts
 			(xy 34.29 67.31) (xy 34.29 81.28)
 		)
@@
 	(wire
 		(pts
-			(xy 160.02 67.31) (xy 160.02 124.46)
+			(xy 163.83 64.77) (xy 163.83 119.38)
 		)
 		(stroke
@@
 	(wire
 		(pts
+			(xy 163.83 64.77) (xy 153.67 64.77)
+		)
+		(stroke
+			(width 0)
+			(type default)
+		)
+	)
+	(wire
+		(pts
 			(xy 199.39 60.96) (xy 201.93 60.96)
 		)
@@
 		(pts
 			(xy 163.83 119.38) (xy 163.83 127)
+		)
+		(stroke
+			(width 0)
+			(type default)
+		)
+	)
+	(wire
+		(pts
+			(xy 160.02 62.23) (xy 153.67 62.23)
 		)
 		(stroke
@@
 	(symbol
 		(lib_id "Device:R_Small_US")
-		(at 151.13 69.85 0)
+		(at 151.13 64.77 0)
 		(unit 1)
 		(exclude_from_sim no)
@@
 		(dnp no)
 		(property "Reference" "R7"
-			(at 152.908 69.088 0)
+			(at 152.908 64.008 0)
 			(effects
 				(font
@@
 		)
 		(property "Value" "0R"
-			(at 155.448 69.088 0)
+			(at 155.448 64.008 0)
 			(effects
 				(font
@@
 		)
 		(property "Footprint" "Resistor_SMD:R_0603_1608Metric"
-			(at 151.13 69.85 0)
+			(at 151.13 64.77 0)
 			(effects
 				(font
@@
 		)
 		(property "Datasheet" "~"
-			(at 151.13 69.85 0)
+			(at 151.13 64.77 0)
 			(effects
 				(font
@@
 		)
 		(property "Description" "Resistor, small US symbol"
-			(at 151.13 69.596 0)
+			(at 151.13 64.516 0)
 			(effects
 				(font
@@
 	(symbol
 		(lib_id "Custom_Parts:5002")
-		(at 153.67 64.77 0)
+		(at 153.67 69.85 0)
 		(unit 1)
 		(exclude_from_sim no)
@@
 		(dnp no)
 		(property "Reference" "TP1"
-			(at 151.638 64.262 0)
+			(at 151.638 69.342 0)
 			(effects
 				(font
@@
 		)
 		(property "Value" "5002"
-			(at 156.21 64.77 0)
+			(at 156.21 69.85 0)
 			(effects
 				(font
@@
 		)
 		(property "Footprint" "Custom_Parts:5002"
-			(at 153.67 64.77 0)
+			(at 153.67 69.85 0)
 			(effects
 				(font
@@
 		)
 		(property "Datasheet" ""
-			(at 153.67 64.77 0)
+			(at 153.67 69.85 0)
 			(effects
 				(font
@@
 		)
 		(property "Description" "TestPoint"
-			(at 153.67 64.77 0)
+			(at 153.67 69.85 0)
 			(effects
 				(font
@@
 		)
 		(property "PARTREV" "H"
-			(at 153.67 64.77 0)
+			(at 153.67 69.85 0)
 			(effects
 				(font
@@
 		)
 		(property "STANDARD" "Manufacturer Recommendations"
-			(at 153.67 64.77 0)
+			(at 153.67 69.85 0)
 			(effects
 				(font
@@
 		)
 		(property "SNAPEDA_PN" "5000"
-			(at 153.67 64.77 0)
+			(at 153.67 69.85 0)
 			(effects
 				(font
@@
 		)
 		(property "MAXIMUM_PACKAGE_HEIGHT" "4.57 mm"
-			(at 153.67 64.77 0)
+			(at 153.67 69.85 0)
 			(effects
 				(font
@@
 		)
 		(property "MANUFACTURER" "Keystone"
-			(at 153.67 64.77 0)
+			(at 153.67 69.85 0)
 			(effects
 				(font
@@
 	(symbol
 		(lib_id "Device:R_Small_US")
-		(at 151.13 67.31 0)
+		(at 151.13 62.23 0)
 		(unit 1)
 		(exclude_from_sim no)
@@
 		(dnp no)
 		(property "Reference" "R8"
-			(at 152.908 66.548 0)
+			(at 152.908 61.468 0)
 			(effects
 				(font
@@
 		)
 		(property "Value" "0R"
-			(at 155.448 66.548 0)
+			(at 155.448 61.468 0)
 			(effects
 				(font
@@
 		)
 		(property "Footprint" "Resistor_SMD:R_0603_1608Metric"
-			(at 151.13 67.31 0)
+			(at 151.13 62.23 0)
 			(effects
 				(font
@@
 		)
 		(property "Datasheet" "~"
-			(at 151.13 67.31 0)
+			(at 151.13 62.23 0)
 			(effects
 				(font
@@
 		)
 		(property "Description" "Resistor, small US symbol"
-			(at 151.13 67.056 0)
+			(at 151.13 61.976 0)
 			(effects
 				(font
@@
 	(symbol
 		(lib_id "Custom_Parts:5002")
-		(at 153.67 62.23 0)
+		(at 153.67 67.31 0)
 		(unit 1)
 		(exclude_from_sim no)
@@
 		(dnp no)
 		(property "Reference" "TP2"
-			(at 151.638 61.722 0)
+			(at 151.638 66.802 0)
 			(effects
 				(font
@@
 		)
 		(property "Value" "5002"
-			(at 156.21 62.23 0)
+			(at 156.21 67.31 0)
 			(effects
 				(font
@@
 		)
 		(property "Footprint" "Custom_Parts:5002"
-			(at 153.67 62.23 0)
+			(at 153.67 67.31 0)
 			(effects
 				(font
@@
 		)
 		(property "Datasheet" ""
-			(at 153.67 62.23 0)
+			(at 153.67 67.31 0)
 			(effects
 				(font
@@
 		)
 		(property "Description" "TestPoint"
-			(at 153.67 62.23 0)
+			(at 153.67 67.31 0)
 			(effects
 				(font
@@
 		)
 		(property "PARTREV" "H"
-			(at 153.67 62.23 0)
+			(at 153.67 67.31 0)
 			(effects
 				(font
@@
 		)
 		(property "STANDARD" "Manufacturer Recommendations"
-			(at 153.67 62.23 0)
+			(at 153.67 67.31 0)
 			(effects
 				(font
@@
 		)
 		(property "SNAPEDA_PN" "5000"
-			(at 153.67 62.23 0)
+			(at 153.67 67.31 0)
 			(effects
 				(font
@@
 		)
 		(property "MAXIMUM_PACKAGE_HEIGHT" "4.57 mm"
-			(at 153.67 62.23 0)
+			(at 153.67 67.31 0)
 			(effects
 				(font
@@
 		)
 		(property "MANUFACTURER" "Keystone"
-			(at 153.67 62.23 0)
-			(effects
-				(font
+			(at 153.67 67.31 0)
+			(effects
+				(font
