File: OPAmp PCB/OPAmp PCB.kicad_sch (KiCad schematic)
At the start: 20 parts, among them J1 Screw_Terminal_01x02, J2 Screw_Terminal_01x02, U1 LM386, U2 LM386, U3 LM386

Commit message: Finished Schematic draft 1
Parts:
- added C10, C11, C12, C9: 470μ, Capacitor_THT:CP_Radial_D10.0mm_P7.50mm, symbol Device:C_Small_US
- added D1: LED, LED_THT:LED_D3.0mm, symbol Device:LED
- added J3: +9V, TerminalBlock:TerminalBlock_MaiXu_MX126-5.0-02P_1x02_P5.00mm, symbol Connector:Screw_Terminal_01x02
- added J4: Out_L, TerminalBlock:TerminalBlock_MaiXu_MX126-5.0-02P_1x02_P5.00mm, symbol Connector:Screw_Terminal_01x02
- added J5: Out_R, TerminalBlock:TerminalBlock_MaiXu_MX126-5.0-02P_1x02_P5.00mm, symbol Connector:Screw_Terminal_01x02
- added R6: 1k, Resistor_THT:R_Axial_DIN0207_L6.3mm_D2.5mm_P7.62mm_Horizontal, symbol Device:R_Small_US
- added SW1: SW_SPDT, Button_Switch_THT:SW_Slide-03_Wuerth-WS-SLTV_10x2.5x6.4_P2.54mm, symbol Switch:SW_Nidec_CAS-120A1
- C1: footprint (none) -> Capacitor_THT:CP_Radial_D5.0mm_P2.50mm
- C2: renamed from C6; footprint (none) -> Capacitor_THT:CP_Radial_D5.0mm_P2.50mm
- C3: renamed from C2; footprint (none) -> Capacitor_THT:CP_Radial_D4.0mm_P2.00mm
- C4: footprint (none) -> Capacitor_THT:CP_Radial_D4.0mm_P2.00mm
- C5: renamed from C8; footprint (none) -> Capacitor_THT:CP_Radial_D4.0mm_P2.00mm
- C6: renamed from C3; value 0.047μ -> 47n; footprint (none) -> Capacitor_THT:C_Disc_D5.0mm_W2.5mm_P2.50mm
- C7: renamed from C5; value 0.047μ -> 47n; footprint (none) -> Capacitor_THT:C_Disc_D5.0mm_W2.5mm_P2.50mm
- C8: renamed from C7; value 0.047μ -> 47n; footprint (none) -> Capacitor_THT:C_Disc_D5.0mm_W2.5mm_P2.50mm
- J1: value Screw_Terminal_01x02 -> In_L; footprint (none) -> TerminalBlock:TerminalBlock_MaiXu_MX126-5.0-02P_1x02_P5.00mm
- J2: value Screw_Terminal_01x02 -> In_R; footprint (none) -> TerminalBlock:TerminalBlock_MaiXu_MX126-5.0-02P_1x02_P5.00mm
- R1, R2, R3, R4, R5: footprint (none) -> Resistor_THT:R_Axial_DIN0207_L6.3mm_D2.5mm_P7.62mm_Horizontal
- RV1, RV2: footprint (none) -> Potentiometer_THT:Potentiometer_Bourns_3386P_Vertical
- U1, U2, U3: footprint (none) -> Package_DIP:DIP-8_W7.62mm_LongPads
Connections:
- net GND: now also C12.1, J3.1 (Pin_1), R6.2, SW1.1 (C)
- net at R5.1, U3.5: now also C11.2
- net at R3.1, U2.5: now also C10.2
- net at R2.1, U1.5: now also C9.2
- net VDC: now reaches U3.6 (V+)
- net VDC: now also U1.6 (V+), U2.6 (V+), C12.2, D1.A, SW1.3 (A)
- new net: C9.1, J4.1 (Pin_1)
- new net: C10.1, J4.2 (Pin_2), J5.1 (Pin_1)
- new net: J3.2 (Pin_2), SW1.2 (B)
- new net: D1.C, R6.1
- new net: C11.1, J5.2 (Pin_2)
Other:
- moved on the sheet: C3, C4, C5, C6, C7, C8

Commit message: Finished Schematic
Parts:
- R1, R3, R5, R6: footprint Resistor_THT:R_Axial_DIN0207_L6.3mm_D2.5mm_P7.62mm_Horizontal -> Resistor_SMD:R_0402_1005Metric
- R2: value 10 -> 47k; footprint Resistor_THT:R_Axial_DIN0207_L6.3mm_D2.5mm_P7.62mm_Horizontal -> Resistor_SMD:R_0402_1005Metric
- R4: value 47k -> 10; footprint Resistor_THT:R_Axial_DIN0207_L6.3mm_D2.5mm_P7.62mm_Horizontal -> Resistor_SMD:R_0402_1005Metric
Connections:
- net GND: now also R2.1; no longer R4.2
- net at C7.2: now also R4.1; no longer R3.2
- net at C11.2, U3.5: now also R5.2; no longer R5.1
- net at C8.2: now also R5.1; no longer R5.2
- net at C2.2, J2.2 (Pin_2): now also R2.2; no longer R4.1
- net at C10.2, U2.5: now also R4.2; no longer R3.1
- net at C6.2: now also R3.2; no longer R2.2
- net at C9.2, U1.5: now also R3.1; no longer R2.1

Commit message: Finished PCB
Parts:
- R1, R2, R3, R4, R5, R6: footprint Resistor_SMD:R_0402_1005Metric -> Resistor_THT:R_Axial_DIN0207_L6.3mm_D2.5mm_P7.62mm_Horizontal
Connections:
- net VDC: now also D1.1 (A); no longer D1.A
- net at R6.1: now also D1.2 (C); no longer D1.C
Changed lines of the file:
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@@
 			)
 		)
-		(property "Footprint" "Resistor_SMD:R_0402_1005Metric"
+		(property "Footprint" "Resistor_THT:R_Axial_DIN0207_L6.3mm_D2.5mm_P7.62mm_Horizontal"
 			(at 69.85 34.29 0)
 			(effects
@@
 			)
 		)
-		(property "Footprint" "Resistor_SMD:R_0402_1005Metric"
+		(property "Footprint" "Resistor_THT:R_Axial_DIN0207_L6.3mm_D2.5mm_P7.62mm_Horizontal"
 			(at 83.82 138.43 0)
 			(effects
@@
 			)
 		)
-		(property "Footprint" "Resistor_SMD:R_0402_1005Metric"
+		(property "Footprint" "Resistor_THT:R_Axial_DIN0207_L6.3mm_D2.5mm_P7.62mm_Horizontal"
 			(at 83.82 71.12 0)
 			(effects
@@
 	)
 	(symbol
-		(lib_id "Device:LED")
-		(at 69.85 26.67 90)
-		(unit 1)
-		(exclude_from_sim no)
-		(in_bom yes)
-		(on_board yes)
-		(dnp no)
-		(property "Reference" "D1"
-			(at 72.644 25.654 0)
-			(effects
-				(font
-					(size 1.27 1.27)
-				)
-				(justify right)
-			)
-		)
-		(property "Value" "LED"
-			(at 72.644 28.194 90)
-			(effects
-				(font
-					(size 1.27 1.27)
-				)
-				(justify right)
-			)
-		)
-		(property "Footprint" "LED_THT:LED_D3.0mm"
-			(at 69.85 26.67 0)
-			(effects
-				(font
-					(size 1.27 1.27)
-				)
-				(hide yes)
-			)
-		)
-		(property "Datasheet" "~"
-			(at 69.85 26.67 0)
-			(effects
-				(font
-					(size 1.27 1.27)
-				)
-				(hide yes)
-			)
-		)
-		(property "Description" "Light emitting diode"
-			(at 69.85 26.67 0)
-			(effects
-				(font
-					(size 1.27 1.27)
-				)
-				(hide yes)
-			)
-		)
-		(property "Sim.Pins" "1=K 2=A"
-			(at 69.85 26.67 0)
-			(effects
-				(font
-					(size 1.27 1.27)
-				)
-				(hide yes)
-			)
-		)
-		(pin "C"
-		)
-		(pin "A"
-		)
-		(instances
-			(project ""
-				(path "/bb6aea29-3813-4033-85c6-fa5357d5717c"
-					(reference "D1")
-					(unit 1)
-				)
-			)
-		)
-	)
-	(symbol
 		(lib_name "R_Small_US_3")
 		(lib_id "Device:R_Small_US")
@@
 			)
 		)
-		(property "Footprint" "Resistor_SMD:R_0402_1005Metric"
+		(property "Footprint" "Resistor_THT:R_Axial_DIN0207_L6.3mm_D2.5mm_P7.62mm_Horizontal"
 			(at 160.02 71.12 0)
 			(effects
@@
 			)
 		)
-		(property "Datasheet" "~"
+		(property "Datasheet" ""
 			(at 160.02 71.12 0)
 			(effects
@@
 			)
 		)
-		(property "Footprint" "Resistor_SMD:R_0402_1005Metric"
+		(property "Footprint" "Resistor_THT:R_Axial_DIN0207_L6.3mm_D2.5mm_P7.62mm_Horizontal"
 			(at 160.02 134.62 0)
 			(effects
@@
 			)
 		)
-		(property "Datasheet" "~"
+		(property "Datasheet" ""
 			(at 160.02 134.62 0)
 			(effects
@@
 			)
 		)
-		(property "Footprint" "Resistor_SMD:R_0402_1005Metric"
+		(property "Footprint" "Resistor_THT:R_Axial_DIN0207_L6.3mm_D2.5mm_P7.62mm_Horizontal"
 			(at 160.02 96.52 0)
 			(effects
@@
 			)
 		)
-		(property "Datasheet" "~"
+		(property "Datasheet" ""
 			(at 160.02 96.52 0)
 			(effects
@@
 					(unit 1)
 				)
+			)
+		)
+	)
+	(symbol
+		(lib_id "Device:LED")
+		(at 69.85 26.67 90)
+		(unit 1)
+		(exclude_from_sim no)
+		(in_bom yes)
+		(on_board yes)
+		(dnp no)
+		(property "Reference" "D1"
+			(at 72.136 25.654 90)
+			(effects
+				(font
+					(size 1.27 1.27)
+				)
+				(justify right)
+			)
+		)
+		(property "Value" "LED"
+			(at 72.136 28.194 90)
+			(effects
+				(font
+					(size 1.27 1.27)
+				)
+				(justify right)
+			)
+		)
+		(property "Footprint" "LED_THT:LED_D3.0mm"
+			(at 69.85 26.67 0)
+			(effects
+				(font
+					(size 1.27 1.27)
+				)
+				(hide yes)
+			)
+		)
+		(property "Datasheet" "~"
+			(at 69.85 26.67 0)
+			(effects
+				(font
+					(size 1.27 1.27)
+				)
+				(hide yes)
+			)
+		)
+		(property "Description" "Light emitting diode"
+			(at 69.85 26.67 0)
+			(effects
+				(font
+					(size 1.27 1.27)
+				)
+				(hide yes)
+			)
+		)
+		(property "Sim.Pins" "1=K 2=A"
+			(at 69.85 26.67 0)
+			(effects
+				(font
+					(size 1.27 1.27)
+				)
+				(hide yes)
+			)
+		)
+		(pin "1"
+		)
+		(pin "2"
+		)
+		(instances
+			(project ""
+				(path "/bb6aea29-3813-4033-85c6-fa5357d5717c"
+					(reference "D1")
+					(unit 1)
+				)
