File: SpotifyDevice/SpotifyDevice.kicad_pcb (KiCad board)
At the start: 2 copper layers, 105.1 x 86.4 mm, 20 parts, among them U1 ESP32-S3-DevKitC, U2 3.5" SPI TFT Display

Commit message: Started Code testing
Routing:
- net Net-(D3-A): track 0.00 -> 1.77 mm
- net Net-(D2-A): track 0.00 -> 1.77 mm
- net Net-(D6-A): track 0.00 -> 1.77 mm
- net Net-(D5-A): track 0.00 -> 1.77 mm
- net Net-(D4-A): track 0.00 -> 1.77 mm
Changed lines of the file:
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@@
+	)
+	(segment
+		(start 102.925 114.25)
+		(end 102.925 115.9625)
+		(width 0.2)
+		(layer "F.Cu")
+		(net 4)
+	)
+	(segment
+		(start 102.925 115.9625)
+		(end 102.9625 116)
+		(width 0.2)
+		(layer "F.Cu")
+		(net 4)
+	)
+	(segment
+		(start 122.925 114.25)
+		(end 122.925 115.9625)
+		(width 0.2)
+		(layer "F.Cu")
+		(net 5)
+	)
+	(segment
+		(start 122.925 115.9625)
+		(end 122.9625 116)
+		(width 0.2)
+		(layer "F.Cu")
+		(net 5)
+	)
+	(segment
+		(start 142.925 115.9625)
+		(end 142.9625 116)
+		(width 0.2)
+		(layer "F.Cu")
+		(net 6)
+	)
+	(segment
+		(start 142.925 114.25)
+		(end 142.925 115.9625)
+		(width 0.2)
+		(layer "F.Cu")
+		(net 6)
+	)
+	(segment
+		(start 162.925 115.9625)
+		(end 162.9625 116)
+		(width 0.2)
+		(layer "F.Cu")
+		(net 7)
+	)
+	(segment
+		(start 162.925 114.25)
+		(end 162.925 115.9625)
+		(width 0.2)
+		(layer "F.Cu")
+		(net 7)
+	)
+	(segment
+		(start 182.925 115.9625)
+		(end 182.9625 116)
+		(width 0.2)
+		(layer "F.Cu")
+		(net 8)
+	)
+	(segment
+		(start 182.925 114.25)
+		(end 182.925 115.9625)
+		(width 0.2)
+		(layer "F.Cu")
+		(net 8)
 	)
 	(segment
